Commit message: Attach the full Orca hand to Nero and drive the arm from webcam wrist motion.
Use MIT motor limits and the official rest pose, then map MediaPipe image-space
wrist and palm size onto carpals IK so combined recording can move arm and fingers.

File: models/nero_prepared.urdf (robot description, URDF)
Before this commit: robot nero, 9 links, 8 joints
Joints:
- joint joint1: limit lower=-2.687807707 upper=2.687807707 effort=100 velocity=5 -> lower=-2.687807707 upper=2.687807707 effort=24 velocity=5
- joint joint2: limit lower=-1.727876707 upper=1.727876707 effort=100 velocity=5 -> lower=-1.727876707 upper=1.727876707 effort=24 velocity=5
- joint joint3: limit lower=-2.740167707 upper=2.740167707 effort=100 velocity=5 -> lower=-2.740167707 upper=2.740167707 effort=16 velocity=5
- joint joint4: limit lower=-0.9948377075 upper=2.129301707 effort=100 velocity=5 -> lower=-0.9948377075 upper=2.129301707 effort=16 velocity=5
- joint joint5: limit lower=-2.740167707 upper=2.740167707 effort=100 velocity=5 -> lower=-2.740167707 upper=2.740167707 effort=8 velocity=5
- joint joint6: limit lower=-0.7155857075 upper=0.9424787075 effort=100 velocity=5 -> lower=-0.7155857075 upper=0.9424787075 effort=8 velocity=5
- joint joint7: limit lower=-1.553343707 upper=1.553343707 effort=100 velocity=5 -> lower=-1.553343707 upper=1.553343707 effort=8 velocity=5
